Commit message: add lidar and control functionally into gazebo

File: description/gazebo_control.xacro (robot description, xacro)
@@ -1,4 +1,25 @@
 <?xml version="1.0"?>
 <robot xmlns:xacro="http://www.ros.org/wiki/xacro">
+    <!--FRICTION-->
+    <gazebo reference="base_link">
+        <mu1>0.001</mu1>
+        <mu2>0.001</mu2>
+    </gazebo>
+    <gazebo reference="base_to_wheel_front_left">
+        <mu1>0.001</mu1>
+        <mu2>0.001</mu2>
+    </gazebo>
+    <gazebo reference="base_to_wheel_front_right">
+        <mu1>0.001</mu1>
+        <mu2>0.001</mu2>
+    </gazebo>
+    <gazebo reference="base_to_wheel_back_left">
+        <mu1>0.001</mu1>
+        <mu2>0.001</mu2>
+    </gazebo>
+    <gazebo reference="base_to_wheel_back_right">
+        <mu1>0.001</mu1>
+        <mu2>0.001</mu2>
+    </gazebo>
     <gazebo>
         <plugin name="diff_drive" filename="libgazebo_ros_diff_drive.so">
@@ -16,5 +37,5 @@
             <wheel_diameter>0.03</wheel_diameter>
             <max_wheel_torque>200</max_wheel_torque>
-            <max_wheel_acceleration>10.0</max_wheel_acceleration>
+            <max_wheel_acceleration>5.0</max_wheel_acceleration>
             <odometry_frame>odom</odometry_frame>
             <robot_base_frame>base_link</robot_base_frame>

File: description/robot.urdf.xacro (robot description, xacro)
@@ -3,3 +3,5 @@
     <xacro:include filename="robot_core.xacro" />
     <xacro:include filename="gazebo_control.xacro"/>
+    <xacro:include filename="lidar.xacro"/>
+    <xacro:include filename="camera.xacro"/>
 </robot>

File: description/robot_core.xacro (robot description, xacro)
@@ -14,4 +14,7 @@
         <color rgba="0 0 0 1" />
     </material>
+    <material name="red">
+        <color rgba="1 0 0 1" />
+    </material>
 <!-- BASE LINK -->
     <link name="base_link">
@@ -25,18 +28,18 @@
     <link name="chassis">
         <visual>
-            <origin xyz="0 0 0.11"/>
+            <origin xyz="0 0 0.08"/>
             <geometry>
-                <box size="0.4 0.4 0.16"/>
+                <box size="0.4 0.25 0.16"/>
             </geometry>
             <material name="white"/>
         </visual>
         <collision>
-            <origin xyz="0 0 0.11"/>
+            <origin xyz="0 0 0.08"/>
             <geometry>
-                <box size="0.4 0.4 0.16"/>
+                <box size="0.4 0.25 0.16"/>
             </geometry>
         </collision>
-        <xacro:inertial_box mass="0.5" x="0.4" y="0.4" z="0.11">
-            <origin xyz="0 0 0.04" rpy="0 0 0"/>
+        <xacro:inertial_box mass="0.5" x="0.4" y="0.25" z="0.16">
+            <origin xyz="0 0 0.08" rpy="0 0 0"/>
         </xacro:inertial_box>
     </link>
@@ -64,5 +67,5 @@
       <cylinder radius="0.03" length="0.03"/>
     </geometry>
-    <origin xyz="0 0 0" rpy="1.5708 0 0"/> <!-- agar menghadap ke samping -->
+    <origin xyz="0 0 0" rpy="0 0 0"/> <!-- agar menghadap ke samping -->
     <material name="black">
       <color rgba="0 0 0 1"/>
@@ -72,8 +75,9 @@
     <geometry>
       <cylinder radius="0.03" length="0.03"/>
-      <origin xyz="0 0 0" rpy="1.5708 0 0"/>
+      <origin xyz="0 0 0" rpy="0 0 0"/>
     </geometry>
   </collision>
-  <xacro:inertial_cylinder mass="0.1" length="0.04" radius="0.05">
+  <!-- <xacro:inertial_cylinder mass="0.1" length="0.04" radius="0.05"> -->
+  <xacro:inertial_cylinder mass="0.1" length="0.03" radius="0.03">
     <origin xyz="0 0 0" rpy="0 0 0"/>
   </xacro:inertial_cylinder>
@@ -85,6 +89,6 @@
   <parent link="base_link"/>
   <child link="wheel_front_left_link"/>
-  <origin xyz="0.165 0.14 0.03" rpy="0 0 0"/>
-  <axis xyz="0 1 0"/>
+  <origin xyz="0.165 0.14 0" rpy="${pi/2} 0 0"/>
+  <axis xyz="0 0 -1"/>
 </joint>
 <!-- kanan-depan -->
@@ -94,5 +98,5 @@
       <cylinder radius="0.03" length="0.03"/>
     </geometry>
-    <origin xyz="0 0 0" rpy="-1.5708 0 0"/>
+    <origin xyz="0 0 0" rpy="0 0 0"/>
     <material name="black">
       <color rgba="0 0 0 1"/>
@@ -102,8 +106,8 @@
     <geometry>
       <cylinder radius="0.03" length="0.03"/>
-      <origin xyz="0 0 0" rpy="-1.5708 0 0"/>
+      <origin xyz="0 0 0" rpy="0 0 0"/>
     </geometry>
   </collision>
-  <xacro:inertial_cylinder mass="0.1" length="0.04" radius="0.05">
+  <xacro:inertial_cylinder mass="0.1" length="0.03" radius="0.03">
     <origin xyz="0 0 0" rpy="0 0 0"/>
   </xacro:inertial_cylinder>
@@ -115,6 +119,6 @@
   <parent link="base_link"/>
   <child link="wheel_front_right_link"/>
-  <origin xyz="0.165 -0.14 0.03" rpy="0 0 0"/>
-  <axis xyz="0 1 0"/>
+  <origin xyz="0.165 -0.14 0" rpy="${pi/2} 0 0"/>
+  <axis xyz="0 0 -1"/>
 </joint>
 <!-- kiri-belakang -->
@@ -124,5 +128,5 @@
       <cylinder radius="0.03" length="0.03"/>
     </geometry>
-    <origin xyz="0 0 0" rpy="1.5708 0 0"/>
+    <origin xyz="0 0 0" rpy="0 0 0"/>
     <material name="black">
       <color rgba="0 0 0 1"/>
@@ -132,8 +136,8 @@
     <geometry>
       <cylinder radius="0.03" length="0.03"/>
-      <origin xyz="0 0 0" rpy="1.5708 0 0"/>
+      <origin xyz="0 0 0" rpy="0 0 0"/>
     </geometry>
   </collision>
-  <xacro:inertial_cylinder mass="0.1" length="0.04" radius="0.05">
+  <xacro:inertial_cylinder mass="0.1" length="0.03" radius="0.03">
     <origin xyz="0 0 0" rpy="0 0 0"/>
   </xacro:inertial_cylinder>
@@ -145,6 +149,6 @@
   <parent link="base_link"/>
   <child link="wheel_back_left_link"/>
-  <origin xyz="-0.165 0.14 0.03" rpy="0 0 0"/>
-  <axis xyz="0 1 0"/>
+  <origin xyz="-0.165 0.14 0" rpy="${pi/2} 0 0"/>
+  <axis xyz="0 0 -1"/>
 </joint>
 <!-- kanan-belakang -->
@@ -154,5 +158,5 @@
       <cylinder radius="0.03" length="0.03"/>
     </geometry>
-    <origin xyz="0 0 0" rpy="-1.5708 0 0"/>
+    <origin xyz="0 0 0" rpy="0 0 0"/>
     <material name="black">
       <color rgba="0 0 0 1"/>
@@ -162,8 +166,8 @@
     <geometry>
       <cylinder radius="0.03" length="0.03"/>
-      <origin xyz="0 0 0" rpy="-1.5708 0 0"/>
+      <origin xyz="0 0 0" rpy="0 0 0"/>
     </geometry>
   </collision>
-  <xacro:inertial_cylinder mass="0.1" length="0.04" radius="0.05">
+  <xacro:inertial_cylinder mass="0.1" length="0.03" radius="0.03">
     <origin xyz="0 0 0" rpy="0 0 0"/>
   </xacro:inertial_cylinder>
@@ -175,6 +179,6 @@
   <parent link="base_link"/>
   <child link="wheel_back_right_link"/>
-  <origin xyz="-0.165 -0.14 0.03" rpy="0 0 0"/>
-  <axis xyz="0 1 0"/>
+  <origin xyz="-0.165 -0.14 0" rpy="${pi/2} 0 0"/>
+  <axis xyz="0 0 -1"/>
 </joint>
 </robot>

Commit message: adding amcl and slam toolbox function

File: description/gazebo_control.xacro (robot description, xacro)
@@ -2,5 +2,5 @@
 <robot xmlns:xacro="http://www.ros.org/wiki/xacro">
     <!--FRICTION-->
-    <gazebo reference="base_link">
+    <!-- <gazebo reference="base_link">
         <mu1>0.001</mu1>
         <mu2>0.001</mu2>
@@ -21,10 +21,10 @@
         <mu1>0.001</mu1>
         <mu2>0.001</mu2>
-    </gazebo>
+    </gazebo> -->
     <gazebo>
         <plugin name="diff_drive" filename="libgazebo_ros_diff_drive.so">
-            <ros>
+            <!-- <ros>
                 <namespace> </namespace>
-            </ros>
+            </ros> -->
             <num_wheel_pairs>2</num_wheel_pairs>
             <left_joint>base_to_wheel_front_left</left_joint>
@@ -37,5 +37,5 @@
             <wheel_diameter>0.03</wheel_diameter>
             <max_wheel_torque>200</max_wheel_torque>
-            <max_wheel_acceleration>5.0</max_wheel_acceleration>
+            <max_wheel_acceleration>10.0</max_wheel_acceleration>
             <odometry_frame>odom</odometry_frame>
             <robot_base_frame>base_link</robot_base_frame>

File: description/lidar.xacro (robot description, xacro)
@@ -46,5 +46,5 @@
             <plugin name="laser_controller" filename="libgazebo_ros_ray_sensor.so">
                 <ros>
-                    <argument>--ros-args --remap ~/out:=scan</argument>
+                    <argument>~/out:=scan</argument>
                 </ros>
                 <output_type>sensor_msgs/LaserScan</output_type>

File: description/robot.urdf.xacro (robot description, xacro)
@@ -3,6 +3,6 @@
     <xacro:include filename="robot_core.xacro" />
     <!-- gazebo include -->
-    <!-- <xacro:include filename="gazebo_control.xacro"/> -->
-    <xacro:include filename="ros2_control.xacro"/>
+    <xacro:include filename="gazebo_control.xacro"/>
+    <!-- <xacro:include filename="ros2_control.xacro"/> -->
     <xacro:include filename="lidar.xacro"/>
     <!-- camera include -->

File: description/robot_core_old.xacro (robot description, xacro)
@@ -2,18 +2,4 @@
 <robot xmlns:xacro="http://www.ros.org/wiki/xacro">
     <xacro:include filename="inertial_macros.xacro"/>
-    <xacro:property name="chassis_length" value="0.4"/>
-    <xacro:property name="chassis_width" value="0.25"/>
-    <xacro:property name="chassis_height" value="0.16"/>
-    <xacro:property name="chassis_mass" value="1.0"/>
-    <xacro:property name="wheel_radius" value="0.03"/>
-    <xacro:property name="wheel_thickness" value="0.03"/>
-    <xacro:property name="wheel_mass" value="0.05"/>
-    <xacro:property name="wheel_offset_x" value="0.165"/>
-    <xacro:property name="wheel_offset_y" value="0.14"/>
-    <xacro:property name="wheel_offset_z" value="0.01"/>
-    <!-- <xacro:property name="caster_wheel_radius" value="0.01"/>
-    <xacro:property name="caster_wheel_mass" value="0.01"/>
-    <xacro:property name="caster_wheel_offset_x" value="0.075"/>
-    <xacro:property name="caster_wheel_offset_z" value="${wheel_offset_z - wheel_radius + caster_wheel_radius}"/> -->
     <material name="white">
         <color rgba="1 1 1 1" />
@@ -33,11 +19,4 @@
 <!-- BASE LINK -->
     <link name="base_link">
-    </link>
-    <joint name="base_footprint_joint" type="fixed">
-        <parent link="base_link"/>
-        <child link="base_footprint"/>
-        <origin xyz="0 0 0" rpy="0 0 0"/>
-    </joint>
-    <link name="base_footprint">
     </link>
 <!-- CHASSIS  LINK-->
@@ -49,22 +28,22 @@
     <link name="chassis">
         <visual>
-            <origin xyz="0 0 ${chassis_height/2}"/>
+            <origin xyz="0 0 0.08"/>
             <geometry>
-                <box size="${chassis_length} ${chassis_width} ${chassis_height}"/>
+                <box size="0.4 0.25 0.16"/>
             </geometry>
             <material name="white"/>
         </visual>
         <collision>
-            <origin xyz="0 0 ${chassis_height/2}"/>
+            <origin xyz="0 0 0.08"/>
             <geometry>
-                <box size="${chassis_length} ${chassis_width} ${chassis_height}"/>
+                <box size="0.4 0.25 0.16"/>
             </geometry>
         </collision>
-        <xacro:inertial_box mass="0.5" x="${chassis_length}" y="${chassis_width}" z="${chassis_height}">
-            <origin xyz="0 0 ${chassis_height/2}" rpy="0 0 0"/>
+        <xacro:inertial_box mass="0.01" x="0.4" y="0.25" z="0.16">
+            <origin xyz="0 0 0.08" rpy="0 0 0"/>
         </xacro:inertial_box>
     </link>
     <gazebo reference="chassis">
-        <material>Gazebo/Orange</material>
+        <material>Gazebo/White</material>
     </gazebo>
 <!-- LEFT FRONT WHEEL -->
@@ -86,6 +65,6 @@
   <visual>
     <geometry>
-      <!-- <sphere radius="${wheel_radius}"/> -->
-      <cylinder radius="${wheel_radius}" length="${wheel_thickness}"/>
+      <sphere radius="0.03"/>
+      <!-- <cylinder radius="0.03" length="0.03"/> -->
     </geometry>
     <origin xyz="0 0 0" rpy="0 0 0"/> <!-- agar menghadap ke samping -->
@@ -96,5 +75,5 @@
   <collision>
     <geometry>
-      <sphere radius="${wheel_radius}"/>
+      <sphere radius="0.03"/>
       <origin xyz="0 0 0" rpy="0 0 0"/>
     </geometry>
@@ -109,5 +88,5 @@
   </collision>
   <!-- <xacro:inertial_cylinder mass="0.1" length="0.04" radius="0.05"> -->
-  <xacro:inertial_cylinder mass="${wheel_mass}" length="${wheel_thickness}" radius="${wheel_radius}">
+  <xacro:inertial_cylinder mass="0.01" length="0.03" radius="0.03">
     <origin xyz="0 0 0" rpy="0 0 0"/>
   </xacro:inertial_cylinder>
@@ -119,6 +98,6 @@
   <parent link="base_link"/>
   <child link="wheel_front_left_link"/>
-  <origin xyz="${wheel_offset_x} ${wheel_offset_y} 0" rpy="-${pi/2} 0 0"/>
-  <axis xyz="0 0 1"/>
+  <origin xyz="0.165 0.14 0" rpy="${pi/2} 0 0"/>
+  <axis xyz="0 0 -1"/>
 </joint>
 <!-- kanan-depan -->
@@ -126,27 +105,27 @@
   <visual>
     <geometry>
-      <!-- <sphere radius="${wheel_radius}"/> -->
-      <cylinder radius="${wheel_radius}" length="${wheel_thickness}"/>
-    </geometry>
-    <origin xyz="0 0 0" rpy="0 0 0"/>
-    <material name="black">
-      <color rgba="0 0 0 1"/>
-    </material>
-  </visual>
-  <collision>
-    <geometry>
-      <sphere radius="${wheel_radius}"/>
-      <origin xyz="0 0 0" rpy="0 0 0"/>
-    </geometry>
-    <friction>
-      <ode>
-        <mu>1000000</mu>
-        <mu2>1000000</mu2>
-        <slip1>0.01</slip1>
-        <slip2>0.01</slip2>
-      </ode>
-    </friction>
-  </collision>
-  <xacro:inertial_cylinder mass="${wheel_mass}" length="${wheel_thickness}" radius="${wheel_radius}">
+      <sphere radius="0.03"/>
+      <!-- <cylinder radius="0.03" length="0.03"/> -->
+    </geometry>
+    <origin xyz="0 0 0" rpy="0 0 0"/>
+    <material name="black">
+      <color rgba="0 0 0 1"/>
+    </material>
+  </visual>
+  <collision>
+    <geometry>
+      <sphere radius="0.03"/>
+      <origin xyz="0 0 0" rpy="0 0 0"/>
+    </geometry>
+    <friction>
+      <ode>
+        <mu>1000000</mu>
+        <mu2>1000000</mu2>
+        <slip1>0.01</slip1>
+        <slip2>0.01</slip2>
+      </ode>
+    </friction>
+  </collision>
+  <xacro:inertial_cylinder mass="0.01" length="0.03" radius="0.03">
     <origin xyz="0 0 0" rpy="0 0 0"/>
   </xacro:inertial_cylinder>
@@ -158,5 +137,5 @@
   <parent link="base_link"/>
   <child link="wheel_front_right_link"/>
-  <origin xyz="${wheel_offset_x} ${-wheel_offset_y} 0" rpy="${pi/2} 0 0"/>
+  <origin xyz="0.165 -0.14 0" rpy="${pi/2} 0 0"/>
   <axis xyz="0 0 -1"/>
 </joint>
@@ -165,27 +144,27 @@
   <visual>
     <geometry>
-      <!-- <sphere radius="${wheel_radius}"/> -->
-      <cylinder radius="${wheel_radius}" length="${wheel_thickness}"/>
-    </geometry>
-    <origin xyz="0 0 0" rpy="0 0 0"/>
-    <material name="black">
-      <color rgba="0 0 0 1"/>
-    </material>
-  </visual>
-  <collision>
-    <geometry>
-      <sphere radius="${wheel_radius}"/>
-      <origin xyz="0 0 0" rpy="0 0 0"/>
-    </geometry>
-    <friction>
-      <ode>
-        <mu>1000000</mu>
-        <mu2>1000000</mu2>
-        <slip1>0.01</slip1>
-        <slip2>0.01</slip2>
-      </ode>
-    </friction>
-  </collision>
-  <xacro:inertial_cylinder mass="${wheel_mass}" length="${wheel_thickness}" radius="${wheel_radius}">
+      <sphere radius="0.03"/>
+      <!-- <cylinder radius="0.03" length="0.03"/> -->
+    </geometry>
+    <origin xyz="0 0 0" rpy="0 0 0"/>
+    <material name="black">
+      <color rgba="0 0 0 1"/>
+    </material>
+  </visual>
+  <collision>
+    <geometry>
+      <sphere radius="0.03"/>
+      <origin xyz="0 0 0" rpy="0 0 0"/>
+    </geometry>
+    <friction>
+      <ode>
+        <mu>1000000</mu>
+        <mu2>1000000</mu2>
+        <slip1>0.01</slip1>
+        <slip2>0.01</slip2>
+      </ode>
+    </friction>
+  </collision>
+  <xacro:inertial_cylinder mass="0.01" length="0.03" radius="0.03">
     <origin xyz="0 0 0" rpy="0 0 0"/>
   </xacro:inertial_cylinder>
@@ -197,5 +176,5 @@
   <parent link="base_link"/>
   <child link="wheel_back_left_link"/>
-  <origin xyz="${-wheel_offset_x} ${wheel_offset_y} 0" rpy="${pi/2} 0 0"/>
+  <origin xyz="-0.165 0.14 0" rpy="${pi/2} 0 0"/>
   <axis xyz="0 0 -1"/>
 </joint>
@@ -204,27 +183,27 @@
   <visual>
     <geometry>
-      <!-- <sphere radius="${wheel_radius}"/> -->
-      <cylinder radius="${wheel_radius}" length="${wheel_thickness}"/>
-    </geometry>
-    <origin xyz="0 0 0" rpy="0 0 0"/>
-    <material name="black">
-      <color rgba="0 0 0 1"/>
-    </material>
-  </visual>
-  <collision>
-    <geometry>
-      <sphere radius="${wheel_radius}"/>
-      <origin xyz="0 0 0" rpy="0 0 0"/>
-    </geometry>
-    <friction>
-      <ode>
-        <mu>1000000</mu>
-        <mu2>1000000</mu2>
-        <slip1>0.01</slip1>
-        <slip2>0.01</slip2>
-      </ode>
-    </friction>
-  </collision>
-  <xacro:inertial_cylinder mass="${wheel_mass}" length="${wheel_thickness}" radius="${wheel_radius}">
+    <sphere radius="0.03"/>
+      <!-- <cylinder radius="0.03" length="0.03"/> -->
+    </geometry>
+    <origin xyz="0 0 0" rpy="0 0 0"/>
+    <material name="black">
+      <color rgba="0 0 0 1"/>
+    </material>
+  </visual>
+  <collision>
+    <geometry>
+      <sphere radius="0.03"/>
+      <origin xyz="0 0 0" rpy="0 0 0"/>
+    </geometry>
+    <friction>
+      <ode>
+        <mu>1000000</mu>
+        <mu2>1000000</mu2>
+        <slip1>0.01</slip1>
+        <slip2>0.01</slip2>
+      </ode>
+    </friction>
+  </collision>
+  <xacro:inertial_cylinder mass="0.01" length="0.03" radius="0.03">
     <origin xyz="0 0 0" rpy="0 0 0"/>
   </xacro:inertial_cylinder>
@@ -236,5 +215,5 @@
   <parent link="base_link"/>
   <child link="wheel_back_right_link"/>
-  <origin xyz="${-wheel_offset_x} ${-wheel_offset_y} 0" rpy="${pi/2} 0 0"/>
+  <origin xyz="-0.165 -0.14 0" rpy="${pi/2} 0 0"/>
   <axis xyz="0 0 -1"/>
 </joint>

File: description/ros2_control.xacro (robot description, xacro)
@@ -10,6 +10,6 @@
                 <param name="max">100</param>
             </command_interface>
+            <state_interface name="position"/>
             <state_interface name="velocity"/>
-            <state_interface name="position"/>
         </joint>
         <joint name="base_to_wheel_front_right">
@@ -18,6 +18,6 @@
                 <param name="max">100</param>
             </command_interface>
+            <state_interface name="position"/>
             <state_interface name="velocity"/>
-            <state_interface name="position"/>
         </joint>
         <joint name="base_to_wheel_back_left">
@@ -26,6 +26,6 @@
                 <param name="max">100</param>
             </command_interface>
+            <state_interface name="position"/>
             <state_interface name="velocity"/>
-            <state_interface name="position"/>
         </joint>
         <joint name="base_to_wheel_back_right">
@@ -34,6 +34,6 @@
                 <param name="max">100</param>
             </command_interface>
+            <state_interface name="position"/>
             <state_interface name="velocity"/>
-             <state_interface name="position"/>
             </joint>
     </ros2_control>
