Commit message: adding few packages for IMU

File: description/robot.urdf.xacro (robot description, xacro)
@@ -3,6 +3,6 @@
     <xacro:include filename="robot_core.xacro" />
     <!-- gazebo include -->
-    <xacro:include filename="gazebo_control.xacro"/>
-    <!-- <xacro:include filename="ros2_control.xacro"/> -->
+    <!-- <xacro:include filename="gazebo_control.xacro"/> -->
+    <xacro:include filename="ros2_control.xacro"/>
     <xacro:include filename="lidar.xacro"/>
     <!-- camera include -->

File: description/robot_core.xacro (robot description, xacro)
@@ -10,5 +10,5 @@
     <xacro:property name="wheel_mass" value="0.05"/>
     <xacro:property name="wheel_offset_x" value="0.165"/>
-    <xacro:property name="wheel_offset_y" value="0.14"/>
+    <xacro:property name="wheel_offset_y" value="0.17"/>
     <xacro:property name="wheel_offset_z" value="0.01"/>
     <!-- <xacro:property name="caster_wheel_radius" value="0.01"/>

File: description/robot_core_old.xacro (robot description, xacro)
@@ -2,4 +2,18 @@
 <robot xmlns:xacro="http://www.ros.org/wiki/xacro">
     <xacro:include filename="inertial_macros.xacro"/>
+    <xacro:property name="chassis_length" value="0.335"/>
+    <xacro:property name="chassis_width" value="0.265"/>
+    <xacro:property name="chassis_height" value="0.138"/>
+    <xacro:property name="chassis_mass" value="1.0"/>
+    <xacro:property name="wheel_radius" value="0.033"/>
+    <xacro:property name="wheel_thickness" value="0.026"/>
+    <xacro:property name="wheel_mass" value="0.05"/>
+    <xacro:property name="wheel_offset_x" value="0.226"/>
+    <xacro:property name="wheel_offset_y" value="0.1485"/>
+    <xacro:property name="wheel_offset_z" value="0.01"/>
+    <xacro:property name="caster_wheel_radius" value="0.01"/>
+    <xacro:property name="caster_wheel_mass" value="0.01"/>
+    <xacro:property name="caster_wheel_offset_x" value="0.075"/>
+    <xacro:property name="caster_wheel_offset_z" value="${wheel_offset_z - wheel_radius + caster_wheel_radius}"/>
     <material name="white">
         <color rgba="1 1 1 1" />

File: description/ros2_control.xacro (robot description, xacro)
@@ -1,5 +1,49 @@
 <?xml version="1.0"?>
 <robot xmlns:xacro="http://www.ros.org/wiki/xacro">
-    <ros2_control name="GazeboSystem" type="system">
+    <ros2_control name="RealRobot" type="system">
+        <hardware>
+            <plugin>topic_based_ros2_control/TopicBasedSystem</plugin>
+            <param name="joint_commands_topic">/diff_cont/commands</param>
+            <param name="joint_states_topic">/raw_joint_states</param>
+            <param name="trigger_joint_command_threshold">-1.0</param>
+            <!-- <param name="device">/dev/ttyACM0</param>
+            <param name="timeout_ms">100</param>
+            <param name="baud_rate">115200</param>
+            <param name="encoder_ticks_per_rotation">106</param> -->
+        </hardware>
+        <joint name="base_to_wheel_front_left">
+            <command_interface name="velocity">
+                <!-- <param name="min">-100</param>
+                <param name="max">100</param> -->
+            </command_interface>
+            <state_interface name="position"/>
+            <state_interface name="velocity"/>
+        </joint>
+        <joint name="base_to_wheel_front_right">
+            <command_interface name="velocity">
+                <!-- <param name="min">-100</param> -->
+                <!-- <param name="max">100</param> -->
+            </command_interface>
+            <state_interface name="position"/>
+            <state_interface name="velocity"/>
+        </joint>
+        <joint name="base_to_wheel_back_left">
+            <command_interface name="velocity">
+                <!-- <param name="min">-100</param> -->
+                <!-- <param name="max">100</param> -->
+            </command_interface>
+            <state_interface name="position"/>
+            <state_interface name="velocity"/>
+        </joint>
+        <joint name="base_to_wheel_back_right">
+            <command_interface name="velocity">
+                <!-- <param name="min">-100</param> -->
+                <!-- <param name="max">100</param> -->
+            </command_interface>
+            <state_interface name="position"/>
+            <state_interface name="velocity"/>
+            </joint>
+    </ros2_control>
+    <!-- <ros2_control name="GazeboSystem" type="system">
         <hardware>
             <plugin>gazebo_ros2_control/GazeboSystem</plugin>
@@ -37,15 +81,9 @@
             <state_interface name="velocity"/>
             </joint>
-    </ros2_control>
+    </ros2_control> -->
     <gazebo>
         <plugin name="gazebo_ros2_control" filename="libgazebo_ros2_control.so">
-            <robot_param>robot_description</robot_param>
-            <robot_param_node>robot_state_publisher</robot_param_node>
-            <max_wheel_torque>200</max_wheel_torque>
-            <max_wheel_acceleration>5.0</max_wheel_acceleration>
-            <odometry_frame>odom</odometry_frame>
-            <robot_base_frame>base_link</robot_base_frame>
-            <parameters>$(find navbot)/config/my_controllers.yaml</parameters>
-            <!-- <parameters>$(find navbot)/config/gaz_ros2_ctl_use_sim.yaml</parameters> -->
+            <parameters>$(find articubot_one)/config/my_controllers.yaml</parameters>
+            <!-- <parameters>$(find articubot_one)/config/gaz_ros2_ctl_use_sim.yaml</parameters> -->
         </plugin>
     </gazebo>

Commit message: making a hardware mapping functionality through SLAM

File: description/robot.urdf.xacro (robot description, xacro)
@@ -4,6 +4,8 @@
     <!-- gazebo include -->
     <!-- <xacro:include filename="gazebo_control.xacro"/> -->
-    <xacro:include filename="ros2_control.xacro"/>
+    <!-- <xacro:include filename="ros2_control.xacro"/> -->
+    <xacro:include filename="ros2_control_interface.xacro"/>
     <xacro:include filename="lidar.xacro"/>
+    <!-- <xacro:include filename="lidar_interface.xacro"/> -->
     <!-- camera include -->
     <xacro:include filename="camera.xacro"/>

File: description/robot_core.xacro (robot description, xacro)
@@ -101,6 +101,6 @@
     <friction>
       <ode>
-        <mu>1000000</mu>
-        <mu2>1000000</mu2>
+        <mu>0.5</mu>
+        <mu2>0.5</mu2>
         <slip1>0.01</slip1>
         <slip2>0.01</slip2>
@@ -141,6 +141,6 @@
     <friction>
       <ode>
-        <mu>1000000</mu>
-        <mu2>1000000</mu2>
+        <mu>0.5</mu>
+        <mu2>0.5</mu2>
         <slip1>0.01</slip1>
         <slip2>0.01</slip2>
@@ -180,6 +180,6 @@
     <friction>
       <ode>
-        <mu>1000000</mu>
-        <mu2>1000000</mu2>
+        <mu>0.5</mu>
+        <mu2>0.5</mu2>
         <slip1>0.01</slip1>
         <slip2>0.01</slip2>
@@ -197,6 +197,6 @@
   <parent link="base_link"/>
   <child link="wheel_back_left_link"/>
-  <origin xyz="${-wheel_offset_x} ${wheel_offset_y} 0" rpy="${pi/2} 0 0"/>
-  <axis xyz="0 0 -1"/>
+  <origin xyz="${-wheel_offset_x} ${wheel_offset_y} 0" rpy="-${pi/2} 0 0"/>
+  <axis xyz="0 0 1"/>
 </joint>
 <!-- kanan-belakang -->
@@ -219,6 +219,6 @@
     <friction>
       <ode>
-        <mu>1000000</mu>
-        <mu2>1000000</mu2>
+        <mu>0.5</mu>
+        <mu2>0.5</mu2>
         <slip1>0.01</slip1>
         <slip2>0.01</slip2>

File: description/ros2_control.xacro (robot description, xacro)
@@ -1,49 +1,5 @@
 <?xml version="1.0"?>
 <robot xmlns:xacro="http://www.ros.org/wiki/xacro">
-    <ros2_control name="RealRobot" type="system">
-        <hardware>
-            <plugin>topic_based_ros2_control/TopicBasedSystem</plugin>
-            <param name="joint_commands_topic">/diff_cont/commands</param>
-            <param name="joint_states_topic">/raw_joint_states</param>
-            <param name="trigger_joint_command_threshold">-1.0</param>
-            <!-- <param name="device">/dev/ttyACM0</param>
-            <param name="timeout_ms">100</param>
-            <param name="baud_rate">115200</param>
-            <param name="encoder_ticks_per_rotation">106</param> -->
-        </hardware>
-        <joint name="base_to_wheel_front_left">
-            <command_interface name="velocity">
-                <!-- <param name="min">-100</param>
-                <param name="max">100</param> -->
-            </command_interface>
-            <state_interface name="position"/>
-            <state_interface name="velocity"/>
-        </joint>
-        <joint name="base_to_wheel_front_right">
-            <command_interface name="velocity">
-                <!-- <param name="min">-100</param> -->
-                <!-- <param name="max">100</param> -->
-            </command_interface>
-            <state_interface name="position"/>
-            <state_interface name="velocity"/>
-        </joint>
-        <joint name="base_to_wheel_back_left">
-            <command_interface name="velocity">
-                <!-- <param name="min">-100</param> -->
-                <!-- <param name="max">100</param> -->
-            </command_interface>
-            <state_interface name="position"/>
-            <state_interface name="velocity"/>
-        </joint>
-        <joint name="base_to_wheel_back_right">
-            <command_interface name="velocity">
-                <!-- <param name="min">-100</param> -->
-                <!-- <param name="max">100</param> -->
-            </command_interface>
-            <state_interface name="position"/>
-            <state_interface name="velocity"/>
-            </joint>
-    </ros2_control>
-    <!-- <ros2_control name="GazeboSystem" type="system">
+    <ros2_control name="GazeboSystem" type="system">
         <hardware>
             <plugin>gazebo_ros2_control/GazeboSystem</plugin>
@@ -81,9 +37,21 @@
             <state_interface name="velocity"/>
             </joint>
-    </ros2_control> -->
+    </ros2_control>
     <gazebo>
         <plugin name="gazebo_ros2_control" filename="libgazebo_ros2_control.so">
-            <parameters>$(find articubot_one)/config/my_controllers.yaml</parameters>
+            <parameters>$(find navbot)/config/my_controllers.yaml</parameters>
             <!-- <parameters>$(find articubot_one)/config/gaz_ros2_ctl_use_sim.yaml</parameters> -->
+        </plugin>
+        <plugin name="p3d_base_controller" filename="libgazebo_ros_p3d.so">
+            <ros>
+                <namespace>/</namespace>
+                <!-- <remapping>odom:=odom_perfect</remapping> -->
+            </ros>
+            <body_name>base_link</body_name>
+            <frame_name>odom</frame_name>
+            <update_rate>50.0</update_rate>
+            <xyz_offset>0 0 0</xyz_offset>
+            <rpy_offset>0 0 0</rpy_offset>
+            <gaussian_noise>0.00</gaussian_noise>
         </plugin>
     </gazebo>
