Commit message: adjusting parameters

File: install/navbot/share/navbot/description/gazebo_control.xacro (robot description, xacro)
@@ -32,6 +32,6 @@
             <left_joint>base_to_wheel_back_left</left_joint>
             <right_joint>base_to_wheel_back_right</right_joint>
-            <wheel_separation>0.29</wheel_separation>
-            <wheel_separation>0.29</wheel_separation>
+            <wheel_separation>0.28</wheel_separation>
+            <wheel_separation>0.28</wheel_separation>
             <wheel_diameter>0.03</wheel_diameter>
             <wheel_diameter>0.03</wheel_diameter>

File: install/navbot/share/navbot/description/robot.urdf.xacro (robot description, xacro)
@@ -3,8 +3,9 @@
     <xacro:include filename="robot_core.xacro" />
     <!-- gazebo include -->
-    <!-- <xacro:include filename="gazebo_control.xacro"/> -->
-    <xacro:include filename="ros2_control.xacro"/>
+    <xacro:include filename="gazebo_control.xacro"/>
+    <!-- <xacro:include filename="ros2_control.xacro"/> -->
     <!-- <xacro:include filename="ros2_control_interface.xacro"/> -->
     <xacro:include filename="lidar.xacro"/>
+    <!-- <xacro:include filename="lidar_interface.xacro"/> -->
     <!-- camera include -->
     <xacro:include filename="camera.xacro"/>

File: install/navbot/share/navbot/description/robot_core.xacro (robot description, xacro)
@@ -3,12 +3,12 @@
     <xacro:include filename="inertial_macros.xacro"/>
     <xacro:property name="chassis_length" value="0.4"/>
-    <xacro:property name="chassis_width" value="0.19"/>
+    <xacro:property name="chassis_width" value="0.25"/>
     <xacro:property name="chassis_height" value="0.16"/>
     <xacro:property name="chassis_mass" value="1.0"/>
-    <xacro:property name="wheel_radius" value="0.025"/>
+    <xacro:property name="wheel_radius" value="0.03"/>
     <xacro:property name="wheel_thickness" value="0.03"/>
     <xacro:property name="wheel_mass" value="0.05"/>
-    <xacro:property name="wheel_offset_x" value="0.145"/>
-    <xacro:property name="wheel_offset_y" value="0.145"/> <!--33 offset total-->
+    <xacro:property name="wheel_offset_x" value="0.165"/>
+    <xacro:property name="wheel_offset_y" value="0.17"/>
     <xacro:property name="wheel_offset_z" value="0.01"/>
     <!-- <xacro:property name="caster_wheel_radius" value="0.01"/>
@@ -101,6 +101,6 @@
     <friction>
       <ode>
-        <mu>1000000</mu>
-        <mu2>1000000</mu2>
+        <mu>0.5</mu>
+        <mu2>0.5</mu2>
         <slip1>0.01</slip1>
         <slip2>0.01</slip2>
@@ -119,6 +119,6 @@
   <parent link="base_link"/>
   <child link="wheel_front_left_link"/>
-  <origin xyz="${-wheel_offset_x} ${-wheel_offset_y} 0" rpy="${pi/2} 0 0"/>
-  <axis xyz="0 0 -1"/>
+  <origin xyz="${wheel_offset_x} ${wheel_offset_y} 0" rpy="-${pi/2} 0 0"/>
+  <axis xyz="0 0 1"/>
 </joint>
 <!-- kanan-depan -->
@@ -141,6 +141,6 @@
     <friction>
       <ode>
-        <mu>1000000</mu>
-        <mu2>1000000</mu2>
+        <mu>0.5</mu>
+        <mu2>0.5</mu2>
         <slip1>0.01</slip1>
         <slip2>0.01</slip2>
@@ -180,6 +180,6 @@
     <friction>
       <ode>
-        <mu>1000000</mu>
-        <mu2>1000000</mu2>
+        <mu>0.5</mu>
+        <mu2>0.5</mu2>
         <slip1>0.01</slip1>
         <slip2>0.01</slip2>
@@ -219,6 +219,6 @@
     <friction>
       <ode>
-        <mu>1000000</mu>
-        <mu2>1000000</mu2>
+        <mu>0.5</mu>
+        <mu2>0.5</mu2>
         <slip1>0.01</slip1>
         <slip2>0.01</slip2>
@@ -236,6 +236,6 @@
   <parent link="base_link"/>
   <child link="wheel_back_right_link"/>
-  <origin xyz="${wheel_offset_x} ${wheel_offset_y} 0" rpy="-${pi/2} 0 0"/>
-  <axis xyz="0 0 1"/>
+  <origin xyz="${-wheel_offset_x} ${-wheel_offset_y} 0" rpy="${pi/2} 0 0"/>
+  <axis xyz="0 0 -1"/>
 </joint>
 </robot>
